File: HW2/hw2_433/hw2_sch.sch (EAGLE design)
At the start: 22 parts, among them J1 USB-MB-H

Commit message: Updated board
Connections:
- net D+: now also J1.D+
- net D-: now also J1.D-
- net USBID: now also J1.ID
Changed lines of the file:
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@@
 <label x="-58.42" y="-45.72" size="1.778" layer="95"/>
+</segment>
+<segment>
+<pinref part="J1" gate="G$1" pin="ID"/>
+<wire x1="-78.74" y1="76.2" x2="-66.04" y2="76.2" width="0.1524" layer="91"/>
+<label x="-73.66" y="76.2" size="1.778" layer="95"/>
 </segment>
 </net>
@@
 <label x="0" y="-10.16" size="1.778" layer="95"/>
 </segment>
+<segment>
+<pinref part="J1" gate="G$1" pin="D-"/>
+<wire x1="-78.74" y1="81.28" x2="-66.04" y2="81.28" width="0.1524" layer="91"/>
+<label x="-68.58" y="81.28" size="1.778" layer="95"/>
+</segment>
 </net>
 <net name="D+" class="0">
@@
 <label x="0" y="-15.24" size="1.778" layer="95"/>
 </segment>
+<segment>
+<pinref part="J1" gate="G$1" pin="D+"/>
+<wire x1="-78.74" y1="78.74" x2="-66.04" y2="78.74" width="0.1524" layer="91"/>
+<label x="-68.58" y="78.74" size="1.778" layer="95"/>
+</segment>
 </net>
