File: HW2/hw2_433/hw2_sch.brd (EAGLE design)
At the start: 50 x 50 mm, 22 parts, among them J1 USB-MB-H

Commit message: Gerber files created
Parts:
- moved C6 3.52 mm to (37.8, 45.1), turned to 90 degrees
- moved C5 1.27 mm to (35.3, 18.9)
Routing:
- net +3V3: track 129.0 -> 131.5 mm
- net D+: track 26.8 -> 28.2 mm
- net B4/USER: track 54.0 -> 55.0 mm
Other:
- board text added: "+"
- board text added: "+3V3"
- board text added: "+5V"
- board text added: "A0"
- board text added: "A1"
- board text added: "A4/LED"
- board text added: "B13"
- board text added: "B14"
- board text added: "B15"
- board text added: "B2"
- board text added: "B3"
- board text added: "B4/USER"
- board text added: "B7"
- board text added: "B8"
- board text added: "B9"
- board text added: "GND"
- board text added: "JATLER ME433"
- board text added: "PGC"
- board text added: "PGD"
